File: Board/Libreductioner.kicad_pcb (KiCad board)
At the start: 2 copper layers, 50.2 x 78.9 mm, 38 parts, among them J1 Conn_01x02_Male, J2 Conn_01x02_Male, J3 Conn_01x02_Male, J4 Conn_01x02_Male, J5 Conn_01x02_Male, J6 Conn_01x02_Male, Q1 IRF3205, U1 ATMEGA168A-AU, U2 PC817, U3 PC817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

Commit message: Board optimized
Parts:
- removed REF**: OSHW-Logo2_7.3x6mm_SilkScreen, Symbol:OSHW-Logo2_7.3x6mm_SilkScreen
- added D3: LED, LED_SMD:LED_0805_2012Metric_Pad0.97x1.50mm_HandSolder, F.Cu at (70.4, 76.6)
- added D4: LED, LED_SMD:LED_0805_2012Metric_Pad0.97x1.50mm_HandSolder, F.Cu at (110.9, 105.1)
- added JP2: SolderJumper_2_Bridged, Jumper:SolderJumper-2_P1.3mm_Bridged_RoundedPad1.0x1.5mm, B.Cu at (103.3, 101.5)
- added R11: 10k, Resistor_SMD:R_0805_2012Metric_Pad1.15x1.50mm_HandSolder, F.Cu at (110.9, 101.2)
- added R12: R, Resistor_SMD:R_0805_2012Metric_Pad1.15x1.50mm_HandSolder, B.Cu at (93.2, 104.0)
- added R13: R, Resistor_SMD:R_0805_2012Metric_Pad1.15x1.50mm_HandSolder, B.Cu at (88.8, 102.3)
- added R14: 10k, Resistor_SMD:R_0805_2012Metric_Pad1.15x1.50mm_HandSolder, F.Cu at (75.8, 130.9)
- added R15: 1k, Resistor_SMD:R_0805_2012Metric_Pad1.15x1.50mm_HandSolder, F.Cu at (80.6, 131.1)
- added R9: 1k, Resistor_SMD:R_0805_2012Metric_Pad1.15x1.50mm_HandSolder, F.Cu at (80.8, 76.7)
- D1: value LED_CRGB -> LED_RCGB
- J3, J4: footprint Connector_PinHeader_2.54mm:PinHeader_2x01_P2.54mm_Vertical -> Connector_PinHeader_2.54mm:PinHeader_1x02_P2.54mm_Vertical
- JP1: value SolderJumper_2_Open -> SolderJumper_2_Bridged; footprint Jumper:SolderJumper-2_P1.3mm_Open_RoundedPad1.0x1.5mm -> Jumper:SolderJumper-2_P1.3mm_Bridged_RoundedPad1.0x1.5mm
- P_AVR1: value Conn_01x05 -> Conn_01x06_Female; footprint Pin_Headers:Pin_Header_Straight_1x05_Pitch2.54mm -> Connector_PinSocket_2.54mm:PinSocket_1x06_P2.54mm_Vertical
- R6: value 2.2k -> 10k
- R7: value R -> 10k
- R8: value R -> 1k
- moved J3 55.8 mm to (69.2, 130.8)
- moved D1 31.2 mm to (88.6, 132.7)
- moved R8 26.3 mm to (103.8, 128.9), turned to 270 degrees
- moved R7 25.4 mm to (113.5, 126.7), turned to 270 degrees
- moved J4 24.5 mm to (69.5, 97.9), turned to 90 degrees
- moved U2 16.0 mm to (107.3, 102.7)
- moved R5 13.7 mm to (82.9, 97.2), turned to 180 degrees
- moved P_AVR1 13.3 mm to (69.3, 134.6), turned to 90 degrees
- moved U3 12.8 mm to (86.5, 99.2), turned to 0 degrees
- moved C8 11.2 mm to (83.3, 105.9)
- moved U4 11.2 mm to (77.2, 104.1)
- moved C9 11.2 mm to (71.5, 104.8)
- moved JP1 8.75 mm to (74.4, 96.1), turned to 90 degrees
- moved J1 7.76 mm to (76.7, 77.1)
- moved R6 7.12 mm to (75.5, 94.2), turned to 0 degrees
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Connections:
- C6 pad 2: /GND12V -> GND
- C7 pad 2: /GND12V -> GND
- C8 pad 2: /GND12V -> GND
- C9 pad 2: /GND12V -> GND
- D1 pad 1: GND -> /D12/MISO
- D1 pad 2: /D10 -> GND
- D1 pad 4: /D12/MISO -> /D10
- J1 pad 1: Net-(J1-Pad1) -> /BUFFERED12V
- J1 pad 2: Net-(J1-Pad2) -> Net-(D2-Pad2)
- J2 pad 1: /GND12V -> GND
- J3 pad 1: /BUFFERED12V -> GND
- J3 pad 2: Net-(J1-Pad1) -> Net-(J3-Pad2)
- J4 pad 1: Net-(J1-Pad2) -> GND
- J4 pad 2: Net-(D2-Pad2) -> VCC
- J5 pad 1: Net-(J1-Pad1) -> /BUFFERED12V
- J5 pad 2: Net-(J1-Pad2) -> Net-(D2-Pad2)
- J6 pad 1: /GND12V -> GND
- JP1 pad 1: GND -> /D9
- JP1 pad 2: /GND12V -> /FET_SIGNAL
- P_AVR1 pad 1: /RESET -> GND
- P_AVR1 pad 2: /D1/TX -> (no net)
- P_AVR1 pad 3: /D0/RX -> VCC
- P_AVR1 pad 4: GND -> /D0/RX
- P_AVR1 pad 5: VCC -> /D1/TX
- Q1 pad 1: Net-(Q1-Pad1) -> /FET_SIGNAL
- Q1 pad 3: /GND12V -> GND
- R5 pad 2: Net-(J1-Pad2) -> Net-(D2-Pad2)
- R6 pad 1: Net-(Q1-Pad1) -> /FET_SIGNAL
- R6 pad 2: /GND12V -> GND
- U2 pad 1: /D6 -> /D2
- U2 pad 3: Net-(Q1-Pad1) -> /FET_SIGNAL
- U2 pad 4: +12V -> /VFET
- U3 pad 2: Net-(J1-Pad1) -> /BUFFERED12V
- U3 pad 4: /D7 -> /D4
- U4 pad 1: /GND12V -> GND
Routing:
- net GND: track 208.7 -> 482.3 mm, vias 2 -> 15
- net /GND12V: track 135.4 -> 0.00 mm, vias 1 -> 0
- net /FET_SIGNAL: track 0.00 -> 42.3 mm, vias 0 -> 4
- net /BUFFERED12V: track 56.2 -> 97.6 mm
- net /D10: track 14.0 -> 54.9 mm
- net /D11/MOSI: track 39.1 -> 76.5 mm
- net /D12/MISO: track 45.3 -> 78.8 mm
- net Net-(D2-Pad2): track 15.8 -> 48.5 mm, vias 0 -> 1
- net +12V: track 62.2 -> 94.5 mm
- net Net-(J1-Pad1): track 32.0 -> 0.00 mm
- net Net-(J1-Pad2): track 27.0 -> 0.00 mm
- net VCC: track 125.9 -> 147.9 mm, vias 3 -> 4
- net /D6: track 23.4 -> 6.57 mm
- net /D2: track 14.9 -> 31.4 mm, vias 1 -> 2
- net Net-(Q1-Pad1): track 16.3 -> 0.00 mm
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- added copper zone on B.Cu, net GND
- added copper zone on F.Cu, net GND
Other:
- board size 50.2 x 78.9 mm -> 50.2 x 73 mm
- board text added: "- +"
- board text added: "Control LED"
- board text added: "IN"
- board text added: "MISO"
- board text added: "MOSI"
- board text added: "NC"
- board text added: "PWR"
- board text added: "Pulldown"
- board text added: "Rev. 1.0 13.05.2018 Andreas Butti"
- board text added: "SCK"
- board text added: "VCC"
- board text added: "Vin"
- board text added: "https://github.com/andreasb242/Libreductioner"
- board text removed: "12V"
- board text removed: "N/C"

Commit message: Board optimisations
Changed lines of the file:
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@@
   )
   (setup
-    (last_trace_width 0.5)
+    (last_trace_width 0.25)
     (user_trace_width 0.5)
     (user_trace_width 1)
@@
     (effects (font (size 0.7 0.7) (thickness 0.1)))
   )
-  (gr_text + (at 112.522 100.076) (layer F.SilkS)
+  (gr_text + (at 112.522 104.013) (layer F.SilkS)
     (effects (font (size 0.7 0.7) (thickness 0.1)))
   )

Commit message: Optimized Board
Parts:
- C2, C3, C4, C5: footprint Capacitors_SMD:C_0805_HandSoldering -> Capacitor_SMD:C_0805_2012Metric_Pad1.15x1.50mm_HandSolder
- U1: footprint Housings_QFP:TQFP-32_7x7mm_Pitch0.8mm -> Package_QFP:TQFP-32_7x7mm_P0.8mm
