File: Board/Libreductioner.sch (KiCad schematic (older format))
At the start: 37 parts, among them J1 Conn_01x02_Male, J2 Conn_01x02_Male, J3 Conn_01x02_Male, J4 Conn_01x02_Male, J5 Conn_01x02_Male, J6 Conn_01x02_Male, Q1 IRF3205, U1 ATMEGA168A-AU, U2 PC817, U3 PC817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

Commit message: Board optimized
Parts:
- removed D1: LED_CRGB, LED_THT:LED_D5.0mm-4, symbol Device:LED_CRGB
- removed JP1: SolderJumper_2_Open, Jumper:SolderJumper-2_P1.3mm_Open_RoundedPad1.0x1.5mm, symbol Jumper:SolderJumper_2_Open
- removed P_AVR1: Conn_01x05, Pin_Headers:Pin_Header_Straight_1x05_Pitch2.54mm, symbol Libreductioner-rescue:Conn_01x05-Connector-Libreductioner-rescue-Libreductioner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
- added D1: LED_RCGB, LED_THT:LED_D5.0mm-4, symbol Device:LED_RCGB
- added D3, D4: LED, LED_SMD:LED_0805_2012Metric_Pad0.97x1.50mm_HandSolder, symbol Device:LED
- added JP1, JP2: SolderJumper_2_Bridged, Jumper:SolderJumper-2_P1.3mm_Bridged_RoundedPad1.0x1.5mm, symbol Jumper:SolderJumper_2_Bridged
- added P_AVR1: Conn_01x06_Female, Connector_PinSocket_2.54mm:PinSocket_1x06_P2.54mm_Vertical, symbol Connector_Generic:Conn_01x06_Female
- added R11, R14: 10k, Resistor_SMD:R_0805_2012Metric_Pad1.15x1.50mm_HandSolder, symbol Device:R
- added R12, R13: R, Resistor_SMD:R_0805_2012Metric_Pad1.15x1.50mm_HandSolder, symbol Device:R
- added R15, R9: 1k, Resistor_SMD:R_0805_2012Metric_Pad1.15x1.50mm_HandSolder, symbol Device:R
- J3, J4: footprint Connector_PinHeader_2.54mm:PinHeader_2x01_P2.54mm_Vertical -> Connector_PinHeader_2.54mm:PinHeader_1x02_P2.54mm_Vertical
- R6: value 2.2k -> 10k
- R7: value R -> 10k
- R8: value R -> 1k
Connections:
- net labels added: FET_SIGNAL, VFET
- net labels removed: GND12V
- wire segments 178 -> 205
- no-connect marks 0 -> 1
Other:
- note added: "5...50mA, Peak 1A\nKeeps induction Voltage away from AVR"
- note added: "FET support 30A at 5V Vds, 100A at 6V Vds"
- note added: "Optional Driver"
- note added: "Optional Resitor, instead of Optocupler"
- note removed: "Power can be completely isolated from Arduino\n(12V may Destroy a PC over USB Port...)"
- moved on the sheet: ISP1, U4

Commit message: Board optimisations
Other:
- note added: "FET support 30A at 5V Vds, 100A at 6V Vds\nAVR Supports 5V, with Optocupler more is possible"
- note removed: "FET support 30A at 5V Vds, 100A at 6V Vds"
Changed lines of the file:
@@
 	1    0    0    -1
 $EndComp
-Text Notes 8550 4850 0    50   ~ 0
-FET support 30A at 5V Vds, 100A at 6V Vds
+Text Notes 8550 4950 0    50   ~ 0
+FET support 30A at 5V Vds, 100A at 6V Vds\nAVR Supports 5V, with Optocupler more is possible
 $EndSCHEMATC

Commit message: Optimized Board
Parts:
- C2, C3, C4, C5: footprint Capacitors_SMD:C_0805_HandSoldering -> Capacitor_SMD:C_0805_2012Metric_Pad1.15x1.50mm_HandSolder
- U1: footprint Housings_QFP:TQFP-32_7x7mm_Pitch0.8mm -> Package_QFP:TQFP-32_7x7mm_P0.8mm
- Y1: footprint Crystals:Crystal_HC18-U_Vertical -> Crystal:Crystal_HC18-U_Vertical
Changed lines of the file:
@@
 F 0 "U1" H 2550 3517 50  0000 C CNN
 F 1 "ATMEGA168A-AU" H 2550 3426 50  0000 C CNN
-F 2 "Housings_QFP:TQFP-32_7x7mm_Pitch0.8mm" H 2500 2150 50  0001 C CIN
+F 2 "Package_QFP:TQFP-32_7x7mm_P0.8mm" H 2500 2150 50  0001 C CIN
 F 3 "http://www.atmel.com/images/atmel-8271-8-bit-avr-microcontroller-atmega48a-48pa-88a-88pa-168a-168pa-328-328p_datasheet.pdf" H 2500 2150 50  0001 C CNN
 	1    2500 2150
@@
 F 0 "C3" H 1515 1946 50  0000 L CNN
 F 1 "100n" H 1515 1855 50  0000 L CNN
-F 2 "Capacitors_SMD:C_0805_HandSoldering" H 1438 1750 50  0001 C CNN
+F 2 "Capacitor_SMD:C_0805_2012Metric_Pad1.15x1.50mm_HandSolder" H 1438 1750 50  0001 C CNN
 F 3 "" H 1400 1900 50  0001 C CNN
 	1    1400 1900
@@
 F 0 "C2" H 1115 1096 50  0000 L CNN
 F 1 "100n" H 1115 1005 50  0000 L CNN
-F 2 "Capacitors_SMD:C_0805_HandSoldering" H 1038 900 50  0001 C CNN
+F 2 "Capacitor_SMD:C_0805_2012Metric_Pad1.15x1.50mm_HandSolder" H 1038 900 50  0001 C CNN
 F 3 "" H 1000 1050 50  0001 C CNN
 	1    1000 1050
@@
 F 0 "Y1" V 4504 1731 50  0000 L CNN
 F 1 "Crystal" V 4595 1731 50  0000 L CNN
-F 2 "Crystals:Crystal_HC18-U_Vertical" H 4550 1600 50  0001 C CNN
+F 2 "Crystal:Crystal_HC18-U_Vertical" H 4550 1600 50  0001 C CNN
 F 3 "" H 4550 1600 50  0001 C CNN
 	1    4550 1600
@@
 F 0 "C4" V 4898 1450 50  0000 C CNN
 F 1 "22n" V 4989 1450 50  0000 C CNN
-F 2 "Capacitors_SMD:C_0805_HandSoldering" H 5188 1300 50  0001 C CNN
+F 2 "Capacitor_SMD:C_0805_2012Metric_Pad1.15x1.50mm_HandSolder" H 5188 1300 50  0001 C CNN
 F 3 "" H 5150 1450 50  0001 C CNN
 	1    5150 1450
@@
 F 0 "C5" V 4898 1750 50  0000 C CNN
 F 1 "22n" V 4989 1750 50  0000 C CNN
-F 2 "Capacitors_SMD:C_0805_HandSoldering" H 5188 1600 50  0001 C CNN
+F 2 "Capacitor_SMD:C_0805_2012Metric_Pad1.15x1.50mm_HandSolder" H 5188 1600 50  0001 C CNN
 F 3 "" H 5150 1750 50  0001 C CNN
 	1    5150 1750

Commit message: Fixed layout bugs found on Testing
Parts:
- added R16, R17, R18: 1k, Resistor_SMD:R_0805_2012Metric_Pad1.15x1.50mm_HandSolder, symbol Device:R
Connections:
- wire segments 205 -> 211
Changed lines of the file:
@@
 Wire Wire Line
 	3050 4450 3050 4550
-Text Label 4100 4450 2    50   ~ 0
+Text Label 4750 4450 2    50   ~ 0
 D11/MOSI
-Text Label 4100 4250 2    50   ~ 0
+Text Label 4750 4250 2    50   ~ 0
 D12/MISO
-Wire Wire Line
-	3600 4250 4100 4250
-Wire Wire Line
-	3600 4450 4100 4450
-Wire Wire Line
-	3600 4650 4100 4650
-Text Label 4100 4650 2    50   ~ 0
+Text Label 4750 4650 2    50   ~ 0
 D10
 $Comp
@@
 Text Label 7150 5150 0    50   ~ 0
 BUFFERED12V
-Wire Wire Line
-	7450 4350 7250 4350
 $Comp
 L power:GND #PWR0102
@@
 Wire Wire Line
 	7750 5150 7150 5150
-Wire Wire Line
-	7750 5150 7750 4550
-Wire Wire Line
-	7750 4550 7250 4550
 Text Label 8550 4700 0    50   ~ 0
 D9
@@
 Text Notes 8550 4950 0    50   ~ 0
 FET support 30A at 5V Vds, 100A at 6V Vds\nAVR Supports 5V, with Optocupler more is possible
+Wire Wire Line
+	4050 4250 4750 4250
+Wire Wire Line
+	4050 4450 4750 4450
+Wire Wire Line
+	4050 4650 4750 4650
+Wire Wire Line
+	3750 4650 3600 4650
+Wire Wire Line
+	3600 4450 3750 4450
+Wire Wire Line
+	3750 4250 3600 4250
+Wire Wire Line
+	7250 4350 7350 4350
+Wire Wire Line
+	7350 4350 7350 4500
+Wire Wire Line
+	7350 4500 7750 4500
+Wire Wire Line
+	7750 4500 7750 5150
+Wire Wire Line
+	7450 4350 7450 4550
+Wire Wire Line
+	7450 4550 7250 4550
+$Comp
+L Device:R R16
+U 1 1 5B129EEC
+P 3900 4250
+F 0 "R16" H 3970 4296 50  0000 L CNN
+F 1 "1k" H 3970 4205 50  0000 L CNN
+F 2 "Resistor_SMD:R_0805_2012Metric_Pad1.15x1.50mm_HandSolder" V 3830 4250 50  0001 C CNN
+F 3 "~" H 3900 4250 50  0001 C CNN
+	1    3900 4250
+	0    1    1    0
+$EndComp
+$Comp
+L Device:R R17
+U 1 1 5B12A029
+P 3900 4450
+F 0 "R17" H 3970 4496 50  0000 L CNN
+F 1 "1k" H 3970 4405 50  0000 L CNN
+F 2 "Resistor_SMD:R_0805_2012Metric_Pad1.15x1.50mm_HandSolder" V 3830 4450 50  0001 C CNN
+F 3 "~" H 3900 4450 50  0001 C CNN
+	1    3900 4450
+	0    1    1    0
+$EndComp
+$Comp
+L Device:R R18
+U 1 1 5B12A0A1
+P 3900 4650
+F 0 "R18" H 3970 4696 50  0000 L CNN
+F 1 "1k" H 3970 4605 50  0000 L CNN
+F 2 "Resistor_SMD:R_0805_2012Metric_Pad1.15x1.50mm_HandSolder" V 3830 4650 50  0001 C CNN
+F 3 "~" H 3900 4650 50  0001 C CNN
+	1    3900 4650
+	0    1    1    0
+$EndComp
 $EndSCHEMATC

Commit message: Board Cleanup, removed all non-needed parts
Parts:
- removed JP1, JP2: SolderJumper_2_Bridged, Jumper:SolderJumper-2_P1.3mm_Bridged_RoundedPad1.0x1.5mm, symbol Jumper:SolderJumper_2_Bridged
- removed R1, R2, R4: R, Resistor_THT:R_Axial_Power_L25.0mm_W6.4mm_P30.48mm, symbol Device:R
- removed R12, R13: R, Resistor_SMD:R_0805_2012Metric_Pad1.15x1.50mm_HandSolder, symbol Device:R
- removed R9: 1k, Resistor_SMD:R_0805_2012Metric_Pad1.15x1.50mm_HandSolder, symbol Device:R
- removed U2: PC817, Package_DIP:DIP-4_W7.62mm, symbol Isolator:PC817
- added D5, D6: LED, LED_SMD:LED_0805_2012Metric_Pad0.97x1.50mm_HandSolder, symbol Device:LED
- C6, C7: value CP -> 1000µF
- R3: value R -> 30Ω
Connections:
- net labels removed: VFET
- wire segments 211 -> 186
Other:
- note added: "12V Input and Power LED"
- note added: "5V Input, if separat powered"
- note added: "5V Regulator for AVR, optional.\nThe AVR / Arduino can be\nseaparate Powered with 5V"
- note added: "AVR, only needed if no Arduino is used"
- note added: "Arduino, no additonal AVR needed"
- note added: "FET support 30A at 5V Vds"
- note added: "Mesuring circuit,\nto measure a Singnal from another generator"
- note added: "User Interface\nRGB LED or 3 standard LEDs"
- note removed: "FET support 30A at 5V Vds, 100A at 6V Vds\nAVR Supports 5V, with Optocupler more is possible"
- note removed: "For Debugging / Configuration"
- note removed: "Optional Driver"
- note removed: "Optional Resitor, instead of Optocupler"
- moved on the sheet: A1, C2, C3, C4, C5, ISP1, Q1, R10, U1, U4, Y1

Commit message: Removed Input: AVR is to slow for measuring the signal precise enough
Parts:
- removed J3: Conn_01x02_Male, Connector_PinHeader_2.54mm:PinHeader_1x02_P2.54mm_Vertical, symbol Connector_Generic:Conn_01x02_Male
- removed R14: 10k, Resistor_SMD:R_0805_2012Metric_Pad1.15x1.50mm_HandSolder, symbol Device:R
- removed R15: 1k, Resistor_SMD:R_0805_2012Metric_Pad1.15x1.50mm_HandSolder, symbol Device:R
- J1, J2, J4, J5, J6: symbol Connector_Generic:Conn_01x02_Male -> Libreductioner-rescue:Conn_01x02_Male-Connector_Generic
- P_AVR1: symbol Connector_Generic:Conn_01x06_Female -> Libreductioner-rescue:Conn_01x06_Female-Connector_Generic
Connections:
- wire segments 186 -> 179
Other:
- note removed: "Mesuring circuit,\nto measure a Singnal from another generator"
Changed lines of the file:
@@
 	10200 4100 10050 4100
 $Comp
-L Connector_Generic:Conn_01x02_Male J1
+L Libreductioner-rescue:Conn_01x02_Male-Connector_Generic J1
 U 1 1 5AFB1F28
 P 9250 6100
@@
 $EndComp
 $Comp
-L Connector_Generic:Conn_01x02_Male J2
+L Libreductioner-rescue:Conn_01x02_Male-Connector_Generic J2
 U 1 1 5B0B6952
 P 8400 1650
@@
 	1000 1750 1000 2100
 $Comp
-L Connector_Generic:Conn_01x02_Male J5
+L Libreductioner-rescue:Conn_01x02_Male-Connector_Generic J5
 U 1 1 5AFD4D2A
 P 9200 6150
@@
 	9200 5900 9250 5900
 $Comp
-L Connector_Generic:Conn_01x02_Male J6
+L Libreductioner-rescue:Conn_01x02_Male-Connector_Generic J6
 U 1 1 5AFE4BC9
 P 8450 1700
@@
 Connection ~ 7100 1450
 $Comp
-L Connector_Generic:Conn_01x06_Female P_AVR1
+L Libreductioner-rescue:Conn_01x06_Female-Connector_Generic P_AVR1
 U 1 1 5AF8AE9E
 P 2150 4450
@@
 	2150 4450 2150 4650
 NoConn ~ 2050 4650
-$Comp
-L Device:R R14
-U 1 1 5B00B932
-P 4100 6450
-F 0 "R14" H 4170 6496 50  0000 L CNN
-F 1 "10k" H 4170 6405 50  0000 L CNN
-F 2 "Resistor_SMD:R_0805_2012Metric_Pad1.15x1.50mm_HandSolder" V 4030 6450 50  0001 C CNN
-F 3 "~" H 4100 6450 50  0001 C CNN
-	1    4100 6450
-	1    0    0    -1
-$EndComp
-$Comp
-L Device:R R15
-U 1 1 5B00B938
-P 4100 6850
-F 0 "R15" H 4170 6896 50  0000 L CNN
-F 1 "1k" H 4170 6805 50  0000 L CNN
-F 2 "Resistor_SMD:R_0805_2012Metric_Pad1.15x1.50mm_HandSolder" V 4030 6850 50  0001 C CNN
-F 3 "~" H 4100 6850 50  0001 C CNN
-	1    4100 6850
-	1    0    0    -1
-$EndComp
-Wire Wire Line
-	4100 6700 4100 6650
-Wire Wire Line
-	4100 6300 4100 6150
-Wire Wire Line
-	4100 7000 4100 7200
-$Comp
-L power:GND #PWR0116
-U 1 1 5B00B941
-P 4100 7200
-F 0 "#PWR0116" H 4100 6950 50  0001 C CNN
-F 1 "GND" H 4105 7027 50  0000 C CNN
-F 2 "" H 4100 7200 50  0001 C CNN
-F 3 "" H 4100 7200 50  0001 C CNN
-	1    4100 7200
-	1    0    0    -1
-$EndComp
-Wire Wire Line
-	4100 6650 3950 6650
-Connection ~ 4100 6650
-Wire Wire Line
-	4100 6650 4100 6600
-Text Label 3950 6650 0    50   ~ 0
-A1
-$Comp
-L Connector_Generic:Conn_01x02_Male J3
-U 1 1 5B016FF4
-P 4200 5950
-F 0 "J3" V 4260 5990 50  0000 L CNN
-F 1 "Conn_01x02_Male" V 4351 5990 50  0000 L CNN
-F 2 "Connector_PinHeader_2.54mm:PinHeader_1x02_P2.54mm_Vertical" H 4200 5950 50  0001 C CNN
-F 3 "~" H 4200 5950 50  0001 C CNN
-	1    4200 5950
-	0    1    1    0
-$EndComp
-Wire Wire Line
-	4200 6150 4600 6150
-Wire Wire Line
-	4600 6150 4600 6550
-$Comp
-L power:GND #PWR0117
-U 1 1 5B021DB4
-P 4600 6550
-F 0 "#PWR0117" H 4600 6300 50  0001 C CNN
-F 1 "GND" H 4605 6377 50  0000 C CNN
-F 2 "" H 4600 6550 50  0001 C CNN
-F 3 "" H 4600 6550 50  0001 C CNN
-	1    4600 6550
-	1    0    0    -1
-$EndComp
 Text Notes 8050 4800 3    50   ~ 0
 5...50mA, Peak 1A\nKeeps induction Voltage away from AVR
 $Comp
-L Connector_Generic:Conn_01x02_Male J4
+L Libreductioner-rescue:Conn_01x02_Male-Connector_Generic J4
 U 1 1 5AFAC480
 P 6400 2850
@@
 Text Notes 6050 2400 0    50   ~ 0
 5V Input, if separat powered
-Wire Notes Line
-	3700 5400 5700 5400
-Wire Notes Line
-	5700 5400 5700 7750
-Wire Notes Line
-	5700 7750 3700 7750
-Wire Notes Line
-	3700 7750 3700 5400
-Text Notes 3750 5600 0    50   ~ 0
-Mesuring circuit,\nto measure a Singnal from another generator
 $Comp
 L Device:LED D3
